File: hardware/2023-24/battery_3.kicad_sch (KiCad schematic)
At the start: 25 parts, among them Q5 BC817, U4 LM5066

Commit message: Pushing for design review
Parts:
- removed C20, C23, C24: C,IEC, symbol PCM_Generic-50:C,IEC
- removed C21, C22: 1u, symbol PCM_Generic-50:C,IEC
- removed D5: D_Zener, symbol Device:D_Zener
- removed D6: D_Schottky, symbol Device:D_Schottky
- removed JP1, JP2, JP3: Jumper_3_Open, symbol Jumper:Jumper_3_Open
- removed Q1, Q2, Q3, Q4: ~, Nexperia:WLCSP-8, symbol Nexperia:GAN3R2-100CBEAZ
- removed Q5: BC817, Package_TO_SOT_SMD:SOT-23, symbol Transistor_BJT:BC817
- removed R10, R11, R12, R13, R15, R16, R8, R9: R_Small_US, symbol Device:R_Small_US
- removed R14: 100k, symbol Device:R_Small_US
- removed U4: LM5066, TI:HTSSOP-28, symbol TI.Library:LM5066
- added C63, C67: 220u, Capacitor_SMD:CP_Elec_18x17.5, symbol PCM_Generic-50:C,IEC
- added C64, C65: 1u, Capacitor_SMD:C_0603_1608Metric, symbol PCM_Generic-50:C,IEC
- added C66: 10n, Capacitor_SMD:C_0402_1005Metric, symbol PCM_Generic-50:C,IEC
- added C68: 30n, Capacitor_SMD:C_0402_1005Metric, symbol PCM_Generic-50:C,IEC
- added D10: 80V, Diode_SMD:D_SMC, symbol Device:D_Schottky
- added D15: 100V, Diode_SMD:D_SOD-123, symbol PCM_Generic-50:D,IEEE
- added D9: 60V, Diode_SMD:D_SMC, symbol Device:D_Zener
- added Q22: NMOS, Package_TO_SOT_SMD:SOT-23-3, symbol Simulation_SPICE:NMOS
- added Q25, Q26, Q27, Q28, Q29, Q30: ~, Nexperia:WLCSP-8, symbol Nexperia:GAN3R2-100CBE
- added Q32: ~, Package_TO_SOT_SMD:SOT-23, symbol Transistor_BJT:BC817
- added Q33: PNP, Package_TO_SOT_SMD:SOT-23-3, symbol Simulation_SPICE:PNP
- added R110, R34, R99: 100k, Resistor_SMD:R_0603_1608Metric, symbol Device:R_Small_US
- added R111: 21.3k, Resistor_SMD:R_0603_1608Metric, symbol Device:R_Small_US
- added R112, R77: 1k, Resistor_SMD:R_0603_1608Metric, symbol Device:R_Small_US
- added R32: 95k, Resistor_SMD:R_0603_1608Metric, symbol Device:R_Small_US
- added R33: 3.9k, Resistor_SMD:R_0603_1608Metric, symbol Device:R_Small_US
- added R79: 33k, Resistor_SMD:R_0603_1608Metric, symbol Device:R_Small_US
- added R82: 10k, Resistor_SMD:R_0603_1608Metric, symbol Device:R_Small_US
- added R84, R85, R90, R91 (x2), R94: 180, Resistor_SMD:R_0603_1608Metric, symbol Device:R_Small_US
- added R89: 500u, Resistor_SMD:R_2512_6332Metric, symbol Device:R_Small_US
- added R92: 56, Resistor_SMD:R_2512_6332Metric, symbol Device:R_Small_US
- added R96: 30, Resistor_SMD:R_2512_6332Metric, symbol Device:R_Small_US
- added R97: 45.3k, Resistor_SMD:R_0603_1608Metric, symbol Device:R_Small_US
- added U16: LM5066, TI:HTSSOP-28, symbol TI.Library:LM5066
Connections:
- net DIODE_B3: now also Q32.1 (B), Q32.3 (C), U16.16 (DIODE)
- net GATE_B3: now also R84.2, R85.2, R90.2, R91.2, R91.2, R92.2, R94.2, R96.1
- net GND: now also C63.2 (-), C64.2 (-), C65.2 (-), C66.2 (-), C67.2 (-), C68.2 (-), D10.2 (A), D9.2 (A), Q22.3 (S), Q32.2 (E), Q33.1 (C), R111.2, R33.1, R79.1, R96.2, R97.1, U16.10 (GND), U16.24 (RETRY), U16.9 (AGND)
- net PGD_B3: now also R99.1, U16.28 (PGD)
- net UVLO/EN_B3: now also Q22.1 (D), R34.2, R79.2, U16.7 (UVLO/EN)
- net VDD_B3: now also U16.20 (ADR0), U16.22 (CL)
- net VIN_B3: now also C63.1 (+), D9.1 (K), R32.2, R34.1, R89.1, U16.4 (VIN_K), U16.5 (VIN)
- net V_SYS: now also C67.1 (+), D10.1 (K), Q25.2 (S), Q26.2 (S), Q27.2 (S), Q28.2 (S), Q29.2 (S), Q30.2 (S), R110.1, U16.1 (OUT)
- new net: C65.1 (+), U16.15 (VREF)
- new net: C68.1 (+), D15.1 (K-), Q33.3 (E)
- new net: Q28.1 (G), R94.1
- new net: Q25.3 (D), Q26.3 (D), Q27.3 (D), Q28.3 (D), Q29.3 (D), Q30.3 (D), R89.2, U16.3 (SENSE)
- new net: R110.2, R111.1, U16.23 (FB)
- new net: Q27.1 (G), R91.1
- new net: Q30.1 (G), R91.1
- new net: R32.1, R33.2, U16.8 (OVLO)
- new net: C64.1 (+), U16.21 (VDD)
- new net: Q22.2 (G), R77.2
- new net: C66.1 (+), U16.25 (TIMER)
- new net: R97.2, U16.26 (PWR)
- new net: Q26.1 (G), R90.1
- new net: Q33.2 (B), R112.1
- new net: Q29.1 (G), R85.1
- new net: Q25.1 (G), R84.1
- new net +3V3: R82.1, R99.2
- new net ALRT_B3: R82.2, U16.14 (SMBA)
- new net EN_B3: R77.1
- new net GATE_OUT_B3: D15.2 (A+), R112.2, R92.1, U16.2 (GATE)
- new net I2C0_SCL: U16.13 (SCLK)
- new net I2C0_SDA: U16.11 (SDAI), U16.12 (SDAO)
- no-connect marks 2 -> 5
Other:
- note added: "ADDR: 0x42"
- company: (none) -> Boise State University
- title: (none) -> Bender 2024 Power Supply
