File: hardware/2023-24/aux_outputs.kicad_sch (KiCad schematic)
At the start: 49 parts, among them Q28 NMOS, Q29 NMOS, Q30 NMOS, U10 ADS1015IDGS, U9 ADS1015IDGS, U9 NCP1117-ADJ_SOT223

Commit message: Hardware ready for design review
Parts:
- removed C17 (x2): 10u, Capacitor_SMD:C_0805_2012Metric, symbol Device:C
- removed C17: 24n, Capacitor_SMD:C_0805_2012Metric, symbol Device:C
- removed R100, R89, R90, R91: 10k, Resistor_SMD:R_0603_1608Metric, symbol Device:R_Small_US
- removed R37: 3.12k, Resistor_SMD:R_0603_1608Metric, symbol Device:R_Small_US
- removed R38: 120, Resistor_SMD:R_0603_1608Metric, symbol Device:R_Small_US
- removed U9: NCP1117-ADJ_SOT223, Package_TO_SOT_SMD:SOT-223-3_TabPin2, symbol Regulator_Linear:NCP1117-ADJ_SOT223
- added J16 (x2), J18 (x3): Conn_01x05_Pin, Connector_PinHeader_2.54mm:PinHeader_1x05_P2.54mm_Vertical_SMD_Pin1Left, symbol Connector:Conn_01x05_Pin
- added R149, R150, R151: 10k, Resistor_SMD:R_0603_1608Metric, symbol Device:R_Small_US
Connections:
- net GND1 is gone; now on net GND: C17.1, C17.1, C17.1, C17.1, C17.1, C17.1, C17.2, C17.2, C17.2, C17.2, R78.2, R79.1, R82.2, R83.1, R94.2, R95.1, U10.3 (GND), U9.1 (ADDR), U9.3 (GND)
- net +5.5V: now also J16.1 (Pin_1), J16.1 (Pin_1)
- net ADC1_RDY: now also J16.4 (Pin_4)
- net ADC2_RDY: now also J16.4 (Pin_4)
- net ALRT_AUX1: now also J18.4 (Pin_4)
- net ALRT_AUX2: now also J18.4 (Pin_4)
- net ALRT_AUX3: now also J18.4 (Pin_4)
- net EN_AUX_1: now also J18.1 (Pin_1)
- net EN_AUX_2: now also J18.1 (Pin_1)
- net EN_AUX_3: now also J18.1 (Pin_1)
- net GND: now also J16.5 (Pin_5), J16.5 (Pin_5), R149.2, R150.2, R151.2
- net I2C1_SCL: now also J16.3 (Pin_3), J16.3 (Pin_3)
- net I2C1_SDA: now also J16.2 (Pin_2), J16.2 (Pin_2)
- net PGD_AUX1: now also J18.5 (Pin_5)
- net PGD_AUX2: now also J18.5 (Pin_5)
- net PGD_AUX3: now also J18.5 (Pin_5)
- net at Q30.2 (G), R99.2: now also R151.1
- net at Q29.2 (G), R92.2: now also R150.1
- net at Q28.2 (G), R76.2: now also R149.1
- new net Aux 1/I2C_SCL: J18.3 (Pin_3)
- new net Aux 1/I2C_SDA: J18.2 (Pin_2)
- new net Aux 2/I2C_SCL: J18.3 (Pin_3)
- new net Aux 2/I2C_SDA: J18.2 (Pin_2)
- new net Aux 3/I2C_SCL: J18.3 (Pin_3)
- new net Aux 3/I2C_SDA: J18.2 (Pin_2)
Other:
- sheet Aux 1 ports: added I2C_SCL, I2C_SDA; removed none
- sheet Aux 2 ports: added I2C_SCL, I2C_SDA; removed none
- sheet Aux 3 ports: added I2C_SCL, I2C_SDA; removed none
- moved on the sheet: Q28, Q29, Q30, R76, R92, R99
