File: hardware/2023-24/battery_1.kicad_sch (KiCad schematic)
At the start: 25 parts, among them Q5 BC817, U4 LM5066

Commit message: Pushing for design review
Parts:
- removed C20: C,IEC, symbol PCM_Generic-50:C,IEC
- removed JP1, JP2, JP3: Jumper_3_Open, symbol Jumper:Jumper_3_Open
- added C30: 220u, Capacitor_SMD:CP_Elec_18x17.5, symbol PCM_Generic-50:C,IEC
- added C31: 30n, Capacitor_SMD:C_0402_1005Metric, symbol PCM_Generic-50:C,IEC
- added D8: 100V, Diode_SMD:D_SOD-123, symbol PCM_Generic-50:D,IEEE
- added Q1, Q2: ~, Nexperia:WLCSP-8, symbol Nexperia:GAN3R2-100CBE
- added Q22: NMOS, Package_TO_SOT_SMD:SOT-23-3, symbol Simulation_SPICE:NMOS
- added Q8: PNP, Package_TO_SOT_SMD:SOT-23-3, symbol Simulation_SPICE:PNP
- added R12, R13, R14, R15, R16, R18: 180, Resistor_SMD:R_0603_1608Metric, symbol Device:R_Small_US
- added R19: 56, Resistor_SMD:R_2512_6332Metric, symbol Device:R_Small_US
- added R20: 30, Resistor_SMD:R_2512_6332Metric, symbol Device:R_Small_US
- added R23, R77: 1k, Resistor_SMD:R_0603_1608Metric, symbol Device:R_Small_US
- added R82 (x3): 10k, Resistor_SMD:R_0603_1608Metric, symbol Device:R_Small_US
- C29: renamed from C24; value C,IEC -> 220u; footprint (none) -> Capacitor_SMD:CP_Elec_18x17.5; MPN (none) -> EEV-FK2A221M
- C32: renamed from C21; footprint (none) -> Capacitor_SMD:C_0603_1608Metric
- C33: renamed from C22; footprint (none) -> Capacitor_SMD:C_0603_1608Metric
- C34: renamed from C23; value C,IEC -> 10n; footprint (none) -> Capacitor_SMD:C_0402_1005Metric
- D7: renamed from D6; value D_Schottky -> 80V; footprint (none) -> Diode_SMD:D_SMC; MPN (none) -> B380-13-F; Manufacturer (none) -> Diodes Inc
- D9: renamed from D5; value D_Zener -> 60V; footprint (none) -> Diode_SMD:D_SMC; MPN (none) -> 5.0SMDJ60A; Manufacturer (none) -> Bourns
- Q3: renamed from Q4; symbol Nexperia:GAN3R2-100CBEAZ -> Nexperia:GAN3R2-100CBE
- Q4: renamed from Q5; value BC817 -> ~; MPN (none) -> MMBT3904T-7-F; Manufacturer (none) -> Diodes Inc
- Q5: renamed from Q3; symbol Nexperia:GAN3R2-100CBEAZ -> Nexperia:GAN3R2-100CBE
- Q6: renamed from Q2; symbol Nexperia:GAN3R2-100CBEAZ -> Nexperia:GAN3R2-100CBE
- Q7: renamed from Q1; symbol Nexperia:GAN3R2-100CBEAZ -> Nexperia:GAN3R2-100CBE
- R17: renamed from R15; value R_Small_US -> 100k; footprint (none) -> Resistor_SMD:R_0603_1608Metric
- R21: renamed from R16; value R_Small_US -> 21.3k; footprint (none) -> Resistor_SMD:R_0603_1608Metric; MPN (none) -> RN73H1JTTD2132B25
- R22: renamed from R8; value R_Small_US -> 500u; footprint (none) -> Resistor_SMD:R_2512_6332Metric; MPN (none) -> WSLP2512L5000FEA
- R24: renamed from R9; value R_Small_US -> 100k; footprint (none) -> Resistor_SMD:R_0603_1608Metric
- R25: renamed from R14; footprint (none) -> Resistor_SMD:R_0603_1608Metric
- R26: renamed from R10; value R_Small_US -> 33k; footprint (none) -> Resistor_SMD:R_0603_1608Metric
- R27: renamed from R11; value R_Small_US -> 95k; footprint (none) -> Resistor_SMD:R_0603_1608Metric
- R29: renamed from R12; value R_Small_US -> 3.9k; footprint (none) -> Resistor_SMD:R_0603_1608Metric
- R33: renamed from R13; value R_Small_US -> 45.3k; footprint (none) -> Resistor_SMD:R_0603_1608Metric
- renumbered U4 to U5
Connections:
- net GND: now also U5.24 (RETRY), C30.2 (-), C31.2 (-), Q22.3 (S), Q8.1 (C), R20.2; no longer U5.14 (SMBA)
- net V_SYS: now also Q3.2 (S), Q5.2 (S), Q6.2 (S), Q7.2 (S), Q1.2 (S), Q2.2 (S); no longer Q3. (S), Q5. (S), Q6. (S), Q7. (S)
- net I2C0_SDA: now reaches U5.11 (SDAI)
- net I2C0_SDA: now also U5.12 (SDAO), R82.2
- net I2C0_SCL: now reaches U5.13 (SCLK)
- net I2C0_SCL: now also R82.2
- net ALRT: now reaches U5.14 (SMBA)
- net ALRT: now also R82.2
- net ADDR2: now reaches U5.18 (ADR2)
- net ADDR1: now reaches U5.19 (ADR1)
- net ADDR0: now reaches U5.20 (ADR0)
- net VDD: now reaches C32.1 (+), U5.21 (VDD)
- net VDD: now also U5.22 (CL)
- net DIODE_B1 renamed DIODE
- removed net GATE_B1: Q3. (S), Q5. (S), Q6. (S), Q7. (S), U5.2 (GATE)
- net PGD_B1 renamed PGD
- net UVLO/EN_B1 renamed UVLO/EN
- net UVLO/EN: now also Q22.1 (D)
- net VDD_B1 renamed +3V3
- net +3V3: now also R82.1, R82.1, R82.1; no longer U5.22 (CL)
- net VIN_B1 renamed VIN
- net VIN: now also C30.1 (+)
- new net: Q2.1 (G), R13.1
- new net: Q5.1 (G), R15.1
- new net: Q22.2 (G), R77.2
- new net: Q1.1 (G), R12.1
- new net: Q6.1 (G), R16.1
- new net: Q8.2 (B), R23.1
- new net: Q7.1 (G), R18.1
- new net: C31.1 (+), D8.1 (K-), Q8.3 (E)
- new net: Q3.1 (G), R14.1
- new net EN: R77.1
- new net GATE: R12.2, R13.2, R14.2, R15.2, R16.2, R18.2, R19.2, R20.1
- new net GATE_OUT: D8.2 (A+), R19.1, R23.2, U5.2 (GATE)
- new net VD: Q1.3 (D), Q2.3 (D), Q3.3 (D), Q5.3 (D), Q6.3 (D), Q7.3 (D), R22.2, U5.3 (SENSE)
- no-connect marks 2 -> 3
Other:
- note added: "ADDR: 0x40"
- moved on the sheet: C29, C32, C33, C34, D7, D9, Q4, R17, R21, R22, R24, R25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

Commit message: Hardware ready for design review
Parts:
- removed R25: 100k, Resistor_SMD:R_0603_1608Metric, symbol Device:R_Small_US
- removed R82 (x3): 10k, Resistor_SMD:R_0603_1608Metric, symbol Device:R_Small_US
- added R77: 10k, Resistor_SMD:R_0603_1608Metric, symbol Device:R_Small_US
Connections:
- net GND: now also R77.2
- net at Q22.2 (G), R77.2: now also R77.1
- net I2C0_SCL renamed I2C_SCL
- net I2C0_SDA renamed I2C_SDA
