File: hardware/2023-24/battery_inputs.kicad_sch (KiCad schematic)
At the start: 20 parts, among them J10 Screw_Terminal_01x01, J11 TBL007A-508-06GY, J2 Conn_01x02, J4 Screw_Terminal_01x01, J5 Screw_Terminal_01x01, J6 Screw_Terminal_01x01, J7 Screw_Terminal_01x01, J8 TBL007A-508-06GY, J9 Screw_Terminal_01x01, K1 G9KB-1A DC12

Commit message: Hardware ready for design review
Parts:
- added J16, J17, J18: Conn_01x05_Pin, Connector_PinHeader_2.54mm:PinHeader_1x05_P2.54mm_Vertical_SMD_Pin1Left, symbol Connector:Conn_01x05_Pin
Connections:
- net ALRT_B1: now also J16.2 (Pin_2)
- net ALRT_B2: now also J17.2 (Pin_2)
- net ALRT_B3: now also J18.2 (Pin_2)
- net EN_B1: now also J16.5 (Pin_5)
- net EN_B2: now also J17.5 (Pin_5)
- net EN_B3: now also J18.5 (Pin_5)
- net PGD_B1: now also J16.1 (Pin_1)
- net PGD_B2: now also J17.1 (Pin_1)
- net PGD_B3: now also J18.1 (Pin_1)
- new net Battery 1/I2C_SCL: J16.3 (Pin_3)
- new net Battery 1/I2C_SDA: J16.4 (Pin_4)
- new net Battery 2/I2C_SCL: J17.3 (Pin_3)
- new net Battery 2/I2C_SDA: J17.4 (Pin_4)
- new net Battery 3/I2C_SCL: J18.3 (Pin_3)
- new net Battery 3/I2C_SDA: J18.4 (Pin_4)
Other:
- sheet Battery 1 ports: added I2C_SCL, I2C_SDA; removed none
- sheet Battery 2 ports: added I2C_SCL, I2C_SDA; removed none
- sheet Battery 3 ports: added I2C_SCL, I2C_SDA; removed none
