File: hardware/2023-24/2023-24_Power_Supply.kicad_pcb (KiCad board)
At the start: 4 copper layers, 325 x 270 mm, 326 parts, among them J1 Conn_02x03_Odd_Even, J10 Screw_Terminal_01x01, J11 TBL007A-508-06GY, J12 Conn_01x02, J13 Screw_Terminal_01x06, J14 Screw_Terminal_01x06, J15 Screw_Terminal_01x06, J2 USB_B_Micro, J3 Conn_01x02, J4 Screw_Terminal_01x01, J5 Screw_Terminal_01x01, J6 Screw_Terminal_01x01, J7 Screw_Terminal_01x01, J8 TBL007A-508-06GY, J9 Screw_Terminal_01x01, K1 G9KB-1A DC12, Q17 PNP, Q18 NMOS, Q26 PNP, Q27 NMOS, Q28 NMOS, Q29 NMOS, Q30 NMOS, Q8 PNP, Q9 NMOS, SW1 SW_MEC_5E, U1 MAX17502G, U10 ADS1015IDGS, U12 LM5066, U14 LM5066, U16 LM5066, U2 RP2040, U3 NCP1117-3.3_SOT223, U4 W25Q128JVS, U5 LM5066, U6 LM5066, U7 LM5066, U8 NCP1117-ADJ_SOT223, U9 ADS1015IDGS, Y1 ABLS-12.000MHZ-B4-T

Commit message: Hardware ready for design review
Parts:
- removed C1, C10, C11, C19, C2, C3, C4, C5, C6, C7: 100n, Capacitor_SMD:C_0402_1005Metric
- removed C12, C13: 2.2u, Capacitor_SMD:C_1210_3225Metric
- removed C14, C8, C9: 1u, Capacitor_SMD:C_0402_1005Metric
- removed C15, C17, C18, C47, C48: 10u, Capacitor_SMD:C_0805_2012Metric
- removed C16: 910p, Capacitor_SMD:C_0402_1005Metric
- removed C20, C21: 27p, Capacitor_SMD:C_0402_1005Metric
- removed C49: 24n, Capacitor_SMD:C_0805_2012Metric
- removed D1, D2, D3, D4: PMEG10030ELPX, Diode_SMD:D_SOD-128
- removed J1: Conn_02x03_Odd_Even, Connector_PinHeader_2.54mm:PinHeader_2x03_P2.54mm_Vertical_SMD
- removed J2: USB_B_Micro, Connector_USB:USB_Micro-B_Wuerth_629105150521_CircularHoles
- removed J3: Conn_01x02, Connector_PinHeader_2.54mm:PinHeader_1x02_P2.54mm_Vertical
- removed L1: 39u, Inductor_SMD:L_12x12mm_H6mm
- removed R1, R2: 27, Resistor_SMD:R_0402_1005Metric
- removed R10, R9: 1k, Capacitor_SMD:C_0402_1005Metric
- removed R100, R114, R131, R146, R30, R31, R32, R52, R7, R72, R89, R90, R91: 10k, Resistor_SMD:R_0603_1608Metric
- removed R109, R126, R141, R25, R47, R67: 100k, Resistor_SMD:R_0603_1608Metric
- removed R3: 100k, Resistor_SMD:R_0402_1005Metric
- removed R4: 3.3M, Resistor_SMD:R_0402_1005Metric
- removed R5: 453k, Resistor_SMD:R_0402_1005Metric
- removed R6: 11.1k, Resistor_SMD:R_0402_1005Metric
- removed R74: 120, Resistor_SMD:R_0603_1608Metric
- removed R75: 3.12k, Resistor_SMD:R_0603_1608Metric
- removed R8: DNP, Capacitor_SMD:C_0402_1005Metric
- removed the REF** at (145.0, 275.0)
- removed the REF** at (145.0, 270.0)
- removed the REF** at (150.0, 280.0)
- removed the REF** at (150.0, 275.0)
- removed the REF** at (150.0, 270.0)
- removed the REF** at (145.0, 280.0)
- removed SW1: SW_MEC_5E, Button_Switch_SMD:SW_Push_1P1T_NO_Vertical_Wuerth_434133025816
- removed U1: MAX17502G, Maxim:TDFN
- removed U2: RP2040, Package_DFN_QFN:QFN-56-1EP_7x7mm_P0.4mm_EP3.2x3.2mm_ThermalVias
- removed U3: NCP1117-3.3_SOT223, Package_TO_SOT_SMD:SOT-223-3_TabPin2
- removed U4: W25Q128JVS, Package_SO:SOIC-8_5.23x5.23mm_P1.27mm
- removed U8: NCP1117-ADJ_SOT223, Package_TO_SOT_SMD:SOT-223-3_TabPin2
- removed Y1: ABLS-12.000MHZ-B4-T, Crystal:Crystal_SMD_Abracon_ABM8G-4Pin_3.2x2.5mm
- added G***: LOGO, Graphics:Bender_Head_44x26, F.Cu at (435.5, 275.0)
- added J16: Conn_01x05_Pin, Connector_PinHeader_2.54mm:PinHeader_1x05_P2.54mm_Vertical_SMD_Pin1Left, F.Cu at (167.0, 170.0)
- added J17: Conn_01x05_Pin, Connector_PinHeader_2.54mm:PinHeader_1x05_P2.54mm_Vertical_SMD_Pin1Left, F.Cu at (255.0, 170.0)
- added J18: Conn_01x05_Pin, Connector_PinHeader_2.54mm:PinHeader_1x05_P2.54mm_Vertical_SMD_Pin1Left, F.Cu at (343.0, 170.0)
- added J20: Conn_01x05_Pin, Connector_PinHeader_2.54mm:PinHeader_1x05_P2.54mm_Vertical_SMD_Pin1Left, F.Cu at (234.0, 236.0)
- added J21: Conn_01x05_Pin, Connector_PinHeader_2.54mm:PinHeader_1x05_P2.54mm_Vertical_SMD_Pin1Left, F.Cu at (322.0, 236.0)
- added J22: Conn_01x05_Pin, Connector_PinHeader_2.54mm:PinHeader_1x05_P2.54mm_Vertical_SMD_Pin1Left, F.Cu at (163.0, 218.0)
- added J23: Conn_01x05_Pin, Connector_PinHeader_2.54mm:PinHeader_1x05_P2.54mm_Vertical_SMD_Pin1Left, F.Cu at (251.0, 218.0)
- added J24: Conn_01x05_Pin, Connector_PinHeader_2.54mm:PinHeader_1x05_P2.54mm_Vertical_SMD_Pin1Left, F.Cu at (339.3, 218.0)
- added R115: 10k, Resistor_SMD:R_0603_1608Metric, F.Cu at (177.0, 161.5)
- added R116: 10k, Resistor_SMD:R_0603_1608Metric, F.Cu at (264.6, 161.5)
- added R148: 10k, Resistor_SMD:R_0603_1608Metric, F.Cu at (352.5, 161.5)
- added R149: 10k, Resistor_SMD:R_0603_1608Metric, F.Cu at (191.0, 212.5)
- added R150: 10k, Resistor_SMD:R_0603_1608Metric, F.Cu at (279.5, 212.5)
- added R151: 10k, Resistor_SMD:R_0603_1608Metric, F.Cu at (367.5, 212.5)
- added REF**: Symbol_HighVoltage_Type2_CopperTop_VerySmall, Symbol:Symbol_HighVoltage_Type2_CopperTop_VerySmall, F.Cu at (232.0, 101.0)
- added REF**: ESD-Logo_8.9x8mm_SilkScreen, Symbol:ESD-Logo_8.9x8mm_SilkScreen, F.Cu at (243.0, 278.0)
- added REF**: Symbol_HighVoltage_Type2_CopperTop_VerySmall, Symbol:Symbol_HighVoltage_Type2_CopperTop_VerySmall, F.Cu at (278.0, 101.0)
- added REF**: ESD-Logo_8.9x8mm_SilkScreen, Symbol:ESD-Logo_8.9x8mm_SilkScreen, F.Cu at (331.5, 278.0)
- added REF**: Symbol_HighVoltage_Type2_CopperTop_VerySmall, Symbol:Symbol_HighVoltage_Type2_CopperTop_VerySmall, F.Cu at (385.0, 101.0)
- added REF**: Symbol_HighVoltage_Type2_CopperTop_VerySmall, Symbol:Symbol_HighVoltage_Type2_CopperTop_VerySmall, F.Cu at (339.0, 101.0)
- K1: value G9KB-1A DC12 -> G9KB-1A-E DC12
- moved R11 45.7 mm to (458.0, 202.0), turned to 0 degrees
- moved C28 45.7 mm to (455.6, 212.0), turned to 0 degrees
- moved C30 35.0 mm to (204.0, 132.0)
- moved C36 35.0 mm to (309.0, 132.0)
- moved C42 35.0 mm to (414.0, 132.0)
- moved D12 35.0 mm to (309.0, 115.5)
- moved D15 35.0 mm to (414.0, 115.5)
- moved D9 35.0 mm to (204.0, 115.5)
- moved J10 35.0 mm to (424.0, 105.0)
- moved J4 35.0 mm to (194.0, 105.0)
- moved J5 35.0 mm to (214.0, 105.0)
- moved J6 35.0 mm to (299.0, 105.0)
- moved J7 35.0 mm to (319.0, 105.0)
- moved J9 35.0 mm to (404.0, 105.0)
- moved J12 34.1 mm to (456.7, 228.0)
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Connections:
- U12 pad 11: I2C1_SDA -> /Aux Outputs/Aux 1/I2C_SDA
- U12 pad 12: I2C1_SDA -> /Aux Outputs/Aux 1/I2C_SDA
- U12 pad 13: I2C1_SCL -> /Aux Outputs/Aux 1/I2C_SCL
- U14 pad 11: I2C1_SDA -> /Aux Outputs/Aux 2/I2C_SDA
- U14 pad 12: I2C1_SDA -> /Aux Outputs/Aux 2/I2C_SDA
- U14 pad 13: I2C1_SCL -> /Aux Outputs/Aux 2/I2C_SCL
- U16 pad 11: I2C1_SDA -> /Aux Outputs/Aux 3/I2C_SDA
- U16 pad 12: I2C1_SDA -> /Aux Outputs/Aux 3/I2C_SDA
- U16 pad 13: I2C1_SCL -> /Aux Outputs/Aux 3/I2C_SCL
- U5 pad 11: I2C0_SDA -> /Battery Switching/Battery 1/I2C_SDA
- U5 pad 12: I2C0_SDA -> /Battery Switching/Battery 1/I2C_SDA
- U5 pad 13: I2C0_SCL -> /Battery Switching/Battery 1/I2C_SCL
- U6 pad 11: I2C0_SDA -> /Battery Switching/Battery 2/I2C_SDA
- U6 pad 12: I2C0_SDA -> /Battery Switching/Battery 2/I2C_SDA
- U6 pad 13: I2C0_SCL -> /Battery Switching/Battery 2/I2C_SCL
- U7 pad 11: I2C0_SDA -> /Battery Switching/Battery 3/I2C_SDA
- U7 pad 12: I2C0_SDA -> /Battery Switching/Battery 3/I2C_SDA
- U7 pad 13: I2C0_SCL -> /Battery Switching/Battery 3/I2C_SCL
Routing:
- net V_SYS: track 311.9 -> 432.2 mm
- net /USB_D_P: track 90.0 -> 0.00 mm
- net /USB_D_N: track 89.9 -> 0.00 mm
- net +3V3: track 51.3 -> 0.00 mm, vias 22 -> 0
- net Net-(D6-K): track 75.2 -> 35.9 mm
- net +9V: track 32.2 -> 0.00 mm, vias 8 -> 0
- net /Aux Outputs/Aux 2/I2C_SCL: track 0.00 -> 30.0 mm
- net /Aux Outputs/Aux 1/I2C_SCL: track 0.00 -> 30.0 mm
- net /Aux Outputs/Aux 3/I2C_SCL: track 0.00 -> 30.0 mm
- net /Aux Outputs/Aux 1/I2C_SDA: track 0.00 -> 28.5 mm
- net /Aux Outputs/Aux 3/I2C_SDA: track 0.00 -> 28.5 mm
- net /Aux Outputs/Aux 2/I2C_SDA: track 0.00 -> 28.5 mm
- net /QSPI_SS: track 25.1 -> 0.00 mm
- net +1V1: track 23.9 -> 0.00 mm, vias 2 -> 0
- net ALRT_AUX3: track 0.00 -> 23.0 mm
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- added copper zone on B.Cu, net (none)
- added copper zone on B.Cu, net GND2
- added copper zone on F.Cu, net V_MOT
- removed copper zone on F.Cu, net +3V3
- removed copper zone on In2.Cu, net +3V3
- removed copper zone on F.Cu, net +9V
- removed copper zone on In2.Cu, net +9V
- removed copper zone on F.Cu, net /+9V_LX
- removed copper zone on F.Cu, net /MCU_REG_IN
- removed copper zone on In1.Cu, net GND
- removed copper zone on In2.Cu, net GND
- removed copper zone on In1.Cu, net GND2
- removed copper zone on In2.Cu, net GND2
Other:
- board size 325 x 270 mm -> 325 x 235 mm
- copper layers 4 -> 2
- board text added: "locked"
- board text removed: "USB_BOOT"

Commit message: Pushing for pre-production review
Changed lines of the file:
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@@
       (plot_on_all_layers_selection 0x0000000_00000000)
       (disableapertmacros false)
-      (usegerberextensions false)
+      (usegerberextensions true)
       (usegerberattributes true)
       (usegerberadvancedattributes true)
-      (creategerberjobfile true)
+      (creategerberjobfile false)
       (dashed_line_dash_ratio 12.000000)
       (dashed_line_gap_ratio 3.000000)
@@
       (plotinvisibletext false)
       (sketchpadsonfab false)
-      (subtractmaskfromsilk false)
+      (subtractmaskfromsilk true)
       (outputformat 1)
       (mirror false)
-      (drillshape 1)
+      (drillshape 0)
       (scaleselection 1)
-      (outputdirectory "")
+      (outputdirectory "gerbers/")
     )
   )
@@
   (segment (start 254.28 212.908909) (end 255.6 211.588909) (width 0.35) (layer "F.Cu") (net 107))
   (segment (start 273.6 211.588909) (end 276.011091 214) (width 0.35) (layer "F.Cu") (net 107))
-  (segment (start 324.4535 245.505) (end 323.9825 245.034) (width 0.25) (layer "F.Cu") (net 108))
   (segment (start 237.15 245.5) (end 236.471 245.5) (width 0.25) (layer "F.Cu") (net 108))
+  (segment (start 325.15 245.5) (end 324.4485 245.5) (width 0.25) (layer "F.Cu") (net 108))
+  (segment (start 324.4485 245.5) (end 323.9825 245.034) (width 0.25) (layer "F.Cu") (net 108))
   (segment (start 323.9825 245.034) (end 323.9825 238.2) (width 0.25) (layer "F.Cu") (net 108))
   (segment (start 236 238.195) (end 236.54 237.655) (width 0.25) (layer "F.Cu") (net 108))
   (segment (start 236.471 245.5) (end 236 245.029) (width 0.25) (layer "F.Cu") (net 108))
-  (segment (start 325.1325 245.505) (end 324.4535 245.505) (width 0.25) (layer "F.Cu") (net 108))
   (segment (start 236 245.029) (end 236 238.195) (width 0.25) (layer "F.Cu") (net 108))
   (segment (start 323.9825 238.2) (end 324.5225 237.66) (width 0.25) (layer "F.Cu") (net 108))
